Commit message: got controls working -- cube listens to rostopics now

File: oars_description/urdf/boat.urdf.xacro (robot description, xacro)
@@ -10,5 +10,5 @@
 		<visual>
 			<geometry>
-				<box size="10 10 10 "/>
+				<box size="1 1 1 "/>
 			</geometry>
 			<material name="white">
@@ -18,11 +18,14 @@
 		<collision>
 			<geometry>
-				<box size="10 10 10 "/>
+				<box size="1 1 1 "/>
 			</geometry>
 		</collision>
 		<inertial>
 			<mass value="1000"/>
-			<box_inertia m="1000" x="10" y="10" z="10"/>
+			<box_inertia m="100" x="1" y="1" z="1"/>
 		</inertial>
 	</link>
+	<gazebo>
+		<plugin name="oars_plugin" filename="liboars_plugin.so"/>
+	</gazebo>
 </robot>
